File: high_power_sym_supply/high_power_sym_supply.sch (KiCad schematic (older format))
At the start: 13 parts, among them J1 ac input, J2 dc output

Commit message: update: add pcb mounting elements to the project
Parts:
- added H1, H2, H3, H4: M3.2, MountingHole:MountingHole_3.2mm_M3, symbol Mechanical:MountingHole
Other:
- note added: "All polarized capacitors: min 63V\nall rest capacitors: min 100V\nall resistor: 0.250W \nLED - standard led diode(red colour)\nGraetz Bridge: with package KB"
- note added: "Mounting elements"
- note removed: "All polarized capacitors: min 63V\nall rest capacitors: min 100V\nLED - standard led diode(red colour)"
Changed lines of the file:
@@
 encoding utf-8
 Sheet 1 1
-Title "AC-DC hight power supply"
+Title "AC/DC high power supply"
 Date "2019-10-05"
 Rev "1.0"
@@
 Text Notes 3150 3350 2    79   ~ 0
 AC input\nmax 2x24V 4A
-Text Notes 7450 4450 0    79   ~ 0
-All polarized capacitors: min 63V\nall rest capacitors: min 100V\nLED - standard led diode(red colour)
+$Comp
+L Mechanical:MountingHole H1
+U 1 1 5D995407
+P 8300 2650
+F 0 "H1" H 8400 2696 50  0000 L CNN
+F 1 "M3.2" H 8400 2605 50  0000 L CNN
+F 2 "MountingHole:MountingHole_3.2mm_M3" H 8300 2650 50  0001 C CNN
+F 3 "~" H 8300 2650 50  0001 C CNN
+	1    8300 2650
+	1    0    0    -1
+$EndComp
+$Comp
+L Mechanical:MountingHole H2
+U 1 1 5D996BC1
+P 8300 2900
+F 0 "H2" H 8400 2946 50  0000 L CNN
+F 1 "M3.2" H 8400 2855 50  0000 L CNN
+F 2 "MountingHole:MountingHole_3.2mm_M3" H 8300 2900 50  0001 C CNN
+F 3 "~" H 8300 2900 50  0001 C CNN
+	1    8300 2900
+	1    0    0    -1
+$EndComp
+$Comp
+L Mechanical:MountingHole H3
+U 1 1 5D996F3B
+P 8750 2650
+F 0 "H3" H 8850 2696 50  0000 L CNN
+F 1 "M3.2" H 8850 2605 50  0000 L CNN
+F 2 "MountingHole:MountingHole_3.2mm_M3" H 8750 2650 50  0001 C CNN
+F 3 "~" H 8750 2650 50  0001 C CNN
+	1    8750 2650
+	1    0    0    -1
+$EndComp
+$Comp
+L Mechanical:MountingHole H4
+U 1 1 5D9971A1
+P 8750 2900
+F 0 "H4" H 8850 2946 50  0000 L CNN
+F 1 "M3.2" H 8850 2855 50  0000 L CNN
+F 2 "MountingHole:MountingHole_3.2mm_M3" H 8750 2900 50  0001 C CNN
+F 3 "~" H 8750 2900 50  0001 C CNN
+	1    8750 2900
+	1    0    0    -1
+$EndComp
+Wire Notes Line
+	8150 2500 8150 3050
+Wire Notes Line
+	8150 3050 9100 3050
+Wire Notes Line
+	9100 3050 9100 2500
+Wire Notes Line
+	9100 2500 8150 2500
+Text Notes 8150 2500 0    59   ~ 0
+Mounting elements
+Text Notes 7550 4800 0    79   ~ 0
+All polarized capacitors: min 63V\nall rest capacitors: min 100V\nall resistor: 0.250W \nLED - standard led diode(red colour)\nGraetz Bridge: with package KB
 $EndSCHEMATC

Commit message: update: I added a more detailed description to the schematic diagram
Other:
- note added: "All polarized capacitors: min 63V\nall rest capacitors: min 100V\nall resistor: 0.250W \nR1, R2 : in range: 2k2...5k6\nresistance depends on output voltage\nLED - standard led diode(red colour)\nGraetz Bridge: with package KB, Vrms : min 35V"
- note removed: "All polarized capacitors: min 63V\nall rest capacitors: min 100V\nall resistor: 0.250W \nLED - standard led diode(red colour)\nGraetz Bridge: with package KB"
Changed lines of the file:
@@
 Mounting elements
 Text Notes 7550 4800 0    79   ~ 0
-All polarized capacitors: min 63V\nall rest capacitors: min 100V\nall resistor: 0.250W \nLED - standard led diode(red colour)\nGraetz Bridge: with package KB
+All polarized capacitors: min 63V\nall rest capacitors: min 100V\nall resistor: 0.250W \nR1, R2 :  in range: 2k2...5k6\nresistance depends on output voltage\nLED - standard led diode(red colour)\nGraetz Bridge: with package KB, Vrms : min 35V
+Wire Notes Line
+	2000 2000 10650 2000
+Wire Notes Line
+	10650 2000 10650 5000
+Wire Notes Line
+	10650 5000 2000 5000
+Wire Notes Line
+	2000 5000 2000 2000
 $EndSCHEMATC
