File: high_power_sym_supply/high_power_sym_supply.kicad_pcb (KiCad board)
At the start: 2 copper layers, 114.3 x 43.2 mm, 13 parts, among them J1 ac input, J2 dc output

Commit message: update: add pcb mounting elements to the project
Parts:
- added H1: M3.2, MountingHole:MountingHole_3.2mm_M3, F.Cu at (78.7, 73.7)
- added H2: M3.2, MountingHole:MountingHole_3.2mm_M3, F.Cu at (78.1, 106.7)
- added H3: M3.2, MountingHole:MountingHole_3.2mm_M3, F.Cu at (182.9, 73.7)
- added H4: M3.2, MountingHole:MountingHole_3.2mm_M3, F.Cu at (182.9, 106.7)
Other:
- board text added: "AC/DC supply AC input: max 2x24V 4A"
- board text removed: "AC/DC supply AC input max 2x24V 4A"
Changed lines of the file:
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@@
     (tracks 54)
     (zones 0)
-    (modules 13)
+    (modules 17)
     (nets 8)
   )
@@
     (visible_elements FFFFFF7F)
     (pcbplotparams
-      (layerselection 0x291fc_fffffffe)
+      (layerselection 0x292fc_fffffffe)
       (usegerberextensions false)
       (usegerberattributes false)
@@
     (add_net "Net-(D2-Pad2)")
     (add_net "Net-(D3-Pad2)")
+  )
+  (module MountingHole:MountingHole_3.2mm_M3 (layer F.Cu)
+    (at 78.74 73.66)
+    (descr "Mounting Hole 3.2mm, no annular, M3")
+    (tags "mounting hole 3.2mm no annular m3")
+    (attr virtual)
+    (fp_text reference H1 (at 0 -4.2) (layer F.SilkS)
+      (effects (font (size 1 1) (thickness 0.15)))
+    )
+    (fp_text value M3.2 (at 0 4.2) (layer F.Fab)
+      (effects (font (size 1 1) (thickness 0.15)))
+    )
+    (fp_circle (center 0 0) (end 3.45 0) (layer F.CrtYd) (width 0.05))
+    (fp_circle (center 0 0) (end 3.2 0) (layer Cmts.User) (width 0.15))
+    (pad 1 np_thru_hole circle (at 0 0) (size 3.2 3.2) (drill 3.2) (layers *.Cu *.Mask))
+  )
+  (module MountingHole:MountingHole_3.2mm_M3 (layer F.Cu)
+    (at 182.88 106.68)
+    (descr "Mounting Hole 3.2mm, no annular, M3")
+    (tags "mounting hole 3.2mm no annular m3")
+    (attr virtual)
+    (fp_text reference H4 (at 0 -4.2) (layer F.SilkS)
+      (effects (font (size 1 1) (thickness 0.15)))
+    )
+    (fp_text value M3.2 (at 0 4.2) (layer F.Fab)
+      (effects (font (size 1 1) (thickness 0.15)))
+    )
+    (fp_circle (center 0 0) (end 3.45 0) (layer F.CrtYd) (width 0.05))
+    (fp_circle (center 0 0) (end 3.2 0) (layer Cmts.User) (width 0.15))
+    (fp_text user %R (at 0.3 0) (layer F.Fab)
+      (effects (font (size 1 1) (thickness 0.15)))
+    )
+    (pad 1 np_thru_hole circle (at 0 0) (size 3.2 3.2) (drill 3.2) (layers *.Cu *.Mask))
+  )
+  (module MountingHole:MountingHole_3.2mm_M3 (layer F.Cu)
+    (at 182.88 73.66)
+    (descr "Mounting Hole 3.2mm, no annular, M3")
+    (tags "mounting hole 3.2mm no annular m3")
+    (attr virtual)
+    (fp_text reference H3 (at 0 -4.2) (layer F.SilkS)
+      (effects (font (size 1 1) (thickness 0.15)))
+    )
+    (fp_text value M3.2 (at 0 4.2) (layer F.Fab)
+      (effects (font (size 1 1) (thickness 0.15)))
+    )
+    (fp_circle (center 0 0) (end 3.45 0) (layer F.CrtYd) (width 0.05))
+    (fp_circle (center 0 0) (end 3.2 0) (layer Cmts.User) (width 0.15))
+    (fp_text user %R (at 0.3 0) (layer F.Fab)
+      (effects (font (size 1 1) (thickness 0.15)))
+    )
+    (pad 1 np_thru_hole circle (at 0 0) (size 3.2 3.2) (drill 3.2) (layers *.Cu *.Mask))
+  )
+  (module MountingHole:MountingHole_3.2mm_M3 (layer F.Cu)
+    (at 78.105 106.68)
+    (descr "Mounting Hole 3.2mm, no annular, M3")
+    (tags "mounting hole 3.2mm no annular m3")
+    (attr virtual)
+    (fp_text reference H2 (at 0 -4.2) (layer F.SilkS)
+      (effects (font (size 1 1) (thickness 0.15)))
+    )
+    (fp_text value M3.2 (at 0 4.2) (layer F.Fab)
+      (effects (font (size 1 1) (thickness 0.15)))
+    )
+    (fp_circle (center 0 0) (end 3.45 0) (layer F.CrtYd) (width 0.05))
+    (fp_circle (center 0 0) (end 3.2 0) (layer Cmts.User) (width 0.15))
+    (fp_text user %R (at 0.3 0) (layer F.Fab)
+      (effects (font (size 1 1) (thickness 0.15)))
+    )
+    (pad 1 np_thru_hole circle (at 0 0) (size 3.2 3.2) (drill 3.2) (layers *.Cu *.Mask))
   )
   (module Capacitor_THT:CP_Radial_D18.0mm_P7.50mm (layer F.Cu)
@@
     (effects (font (size 1 1) (thickness 0.15)))
   )
-  (dimension 43.18 (width 0.15) (layer Dwgs.User)
-    (gr_text "43,180 mm" (at 194.34 90.17 90) (layer Dwgs.User)
+  (dimension 43.18 (width 0.15) (layer Cmts.User)
+    (gr_text "43,180 mm" (at 194.34 90.17 90) (layer Cmts.User)
       (effects (font (size 1 1) (thickness 0.15)))
     )
@@
     (arrow2b (pts (xy 193.04 111.76) (xy 192.453579 110.633496)))
   )
-  (dimension 114.3 (width 0.15) (layer Dwgs.User)
-    (gr_text "114,300 mm" (at 130.81 118.14) (layer Dwgs.User)
+  (dimension 114.3 (width 0.15) (layer Cmts.User)
+    (gr_text "114,300 mm" (at 130.81 118.14) (layer Cmts.User)
       (effects (font (size 1 1) (thickness 0.15)))
     )
@@
     (effects (font (size 2 2) (thickness 0.5)) (justify left))
   )
-  (gr_text "AC/DC supply\nAC input max 2x24V 4A" (at 76.2 73.66) (layer F.SilkS)
-    (effects (font (size 1.5 1.5) (thickness 0.3)) (justify left))
-  )
-  (gr_text "SQ7EQE\nGNU GPLv3\n" (at 87.63 105.41) (layer F.SilkS)
+  (gr_text "AC/DC supply\nAC input:\nmax 2x24V 4A" (at 83.82 73.66) (layer F.SilkS)
+    (effects (font (size 1.2 1.2) (thickness 0.2)) (justify left))
+  )
+  (gr_text "SQ7EQE\nGNU GPLv3\n" (at 92.075 107.95) (layer F.SilkS)
     (effects (font (size 1.5 1.5) (thickness 0.15)) (justify left))
   )
@@
     (effects (font (size 3 3) (thickness 0.4)))
   )
-  (gr_text "-\nGND\n+" (at 185.42 101.6) (layer F.SilkS)
+  (gr_text "-\nGND\n+" (at 179.705 101.6) (layer F.SilkS)
     (effects (font (size 2 2) (thickness 0.4)) (justify right))
   )
-  (gr_text "AC\nGND\nAC" (at 76.2 104.14) (layer F.SilkS)
+  (gr_text "AC\nGND\nAC" (at 81.915 104.14) (layer F.SilkS)
     (effects (font (size 2 2) (thickness 0.4)) (justify left))
   )

Commit message: update: I fixed bugs with the pcb board layout
Parts:
- moved H2 0.63 mm to (78.7, 106.7)
Changed lines of the file:
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@@
     (pad_to_mask_clearance 0.051)
     (solder_mask_min_width 0.25)
-    (aux_axis_origin 0 0)
+    (aux_axis_origin 73.66 111.76)
     (visible_elements FFFFFF7F)
     (pcbplotparams
@@
   )
   (module MountingHole:MountingHole_3.2mm_M3 (layer F.Cu)
-    (at 78.105 106.68)
+    (at 78.74 106.68)
     (descr "Mounting Hole 3.2mm, no annular, M3")
     (tags "mounting hole 3.2mm no annular m3")
