File: keyboard_lab1/keyboard_lab1.kicad_pcb (KiCad board)
At the start: 2 copper layers, 96.5 x 50.8 mm, 9 parts, among them J1 pinout, SW1 SW1, SW2 SW2, SW3 SW3, SW4 SW4, SW5 LEFT, SW6 RIGHT, SW7 UP, SW8 DOWN

Commit message: update: add new usability
Parts:
- added G***: LOGO, keyboard_lab1:instructable, F.Cu at (141.0, 106.7)
