File: microUSB-to-pcb-adapter/microUSB-to-pcb-adapter.kicad_pcb (KiCad board)
At the start: 2 copper layers, 24.1 x 15.2 mm, 2 parts, among them J1 USB_B_Micro, J2 PCB PinHeader

Commit message: update: I have modified a PCB design ...
Other:
- board text added: "D+"
- board text added: "D-"
- board text added: "GND"
- board text added: "ID"
- board text added: "SHIELD"
- board text added: "VBUS"
Changed lines of the file:
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@@
   (general
     (thickness 1.6)
-    (drawings 13)
+    (drawings 19)
     (tracks 26)
     (zones 0)
@@
     (visible_elements FFFFFF7F)
     (pcbplotparams
-      (layerselection 0x3d0fc_ffffffff)
+      (layerselection 0x3d2fc_ffffffff)
       (usegerberextensions false)
       (usegerberattributes true)
@@
       (effects (font (size 1 1) (thickness 0.15)))
     )
-    (fp_text value USB_B_Micro (at 0 4.6 270) (layer F.Fab)
+    (fp_text value USB_B_Micro (at 0 -4.445 270) (layer F.Fab)
       (effects (font (size 1 1) (thickness 0.15)))
     )
@@
     (pad 6 thru_hole oval (at 0 -12.7 90) (size 1.7 1.7) (drill 1) (layers *.Cu *.Mask)
       (net 1 "Net-(J1-Pad6)"))
-    (model ${KISYS3DMOD}/Connector_PinHeader_2.54mm.3dshapes/PinHeader_1x06_P2.54mm_Vertical.wrl
+    (model ${KISYS3DMOD}/Connector_PinHeader_2.54mm.3dshapes/PinHeader_1x06_P2.54mm_Vertical.step
       (at (xyz 0 0 0))
       (scale (xyz 1 1 1))
       (rotate (xyz 0 0 0))
     )
+  )
+  (gr_text SHIELD (at 104.14 88.646 90) (layer F.SilkS)
+    (effects (font (size 1 1) (thickness 0.15)) (justify left))
+  )
+  (gr_text GND (at 106.68 88.646 90) (layer F.SilkS)
+    (effects (font (size 1 1) (thickness 0.15)) (justify left))
+  )
+  (gr_text ID (at 109.22 88.646 90) (layer F.SilkS)
+    (effects (font (size 1 1) (thickness 0.15)) (justify left))
+  )
+  (gr_text D+ (at 111.76 87.376 90) (layer F.SilkS)
+    (effects (font (size 1 1) (thickness 0.15)))
+  )
+  (gr_text D- (at 114.3 88.646 90) (layer F.SilkS)
+    (effects (font (size 1 1) (thickness 0.15)) (justify left))
+  )
+  (gr_text VBUS (at 116.84 88.392 90) (layer F.SilkS)
+    (effects (font (size 1 1) (thickness 0.15)) (justify left))
   )
   (dimension 15.24 (width 0.15) (layer Cmts.User)
@@
     (arrow2b (pts (xy 95.25 95.25) (xy 96.376504 94.663579)))
   )
-  (gr_text "microUSB\nto PCB Adapter\nby SQ7EQE" (at 102.87 82.55) (layer F.SilkS)
-    (effects (font (size 1 1) (thickness 0.15)) (justify left))
+  (gr_text "microUSB to PCB\nAdapter by SQ7EQE" (at 103.632 81.026) (layer F.SilkS)
+    (effects (font (size 1 1) (thickness 0.15) italic) (justify left))
   )
   (gr_line (start 119.38 93.98) (end 95.25 93.98) (layer Edge.Cuts) (width 0.05))
@@
   (gr_line (start 95.25 78.74) (end 119.38 78.74) (layer Edge.Cuts) (width 0.05))
   (gr_line (start 95.25 93.98) (end 95.25 78.74) (layer Edge.Cuts) (width 0.05))
-  (gr_text 6 (at 104.14 88.9) (layer F.SilkS)
-    (effects (font (size 1 1) (thickness 0.15)))
-  )
-  (gr_text 5 (at 106.68 88.9) (layer F.SilkS)
-    (effects (font (size 1 1) (thickness 0.15)))
-  )
-  (gr_text 4 (at 109.22 88.9) (layer F.SilkS)
-    (effects (font (size 1 1) (thickness 0.15)))
-  )
-  (gr_text 3 (at 111.76 88.9) (layer F.SilkS)
-    (effects (font (size 1 1) (thickness 0.15)))
-  )
-  (gr_text 2 (at 114.3 88.9) (layer F.SilkS)
-    (effects (font (size 1 1) (thickness 0.15)))
-  )
-  (gr_text 1 (at 116.84 88.9) (layer F.SilkS)
-    (effects (font (size 1 1) (thickness 0.15)))
-  )
+  (gr_text 6 (at 104.14 89.535) (layer F.SilkS)
+    (effects (font (size 1 1) (thickness 0.15)))
+  )
+  (gr_text 5 (at 106.68 89.535) (layer F.SilkS)
+    (effects (font (size 1 1) (thickness 0.15)))
+  )
+  (gr_text 4 (at 109.22 89.535) (layer F.SilkS)
+    (effects (font (size 1 1) (thickness 0.15)))
+  )
+  (gr_text 3 (at 111.76 89.535) (layer F.SilkS)
+    (effects (font (size 1 1) (thickness 0.15)))
+  )
+  (gr_text 2 (at 114.3 89.535) (layer F.SilkS)
+    (effects (font (size 1 1) (thickness 0.15)))
+  )
+  (gr_text 1 (at 116.84 89.535) (layer F.SilkS)
+    (effects (font (size 1 1) (thickness 0.15)))
+  )
