File: microUSB-to-pcb-power-adapter/microUSB-to-pcb-power-adapter.kicad_pcb (KiCad board)
At the start: 2 copper layers, 22.9 x 10.2 mm, 2 parts, among them J1 Molex_47346-0001, J2 Conn_PinHeader_PCB

Commit message: update: I have re-generate PCB Gerber files
Parts:
- J2: moved to B.Cu
- moved J2 5.08 mm to (119.4, 87.6)
Changed lines of the file:
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@@
   )
   (setup
-    (last_trace_width 0.4)
+    (last_trace_width 0.25)
     (user_trace_width 0.4)
     (trace_clearance 0.2)
@@
     (add_net "Net-(J1-Pad6)")
   )
-  (module microUSB-to-pcb-power-adapter:PinHeader_2x03_P2.54mm_Vertical (layer F.Cu)
-    (at 124.46 87.63 270)
+  (module microUSB-to-pcb-power-adapter:PinHeader_2x03_P2.54mm_Vertical (layer B.Cu)
+    (at 119.38 87.63 270)
     (descr "Through hole straight pin header, 2x03, 2.54mm pitch, double rows")
     (tags "Through hole pin header THT 2x03 2.54mm double row")
-    (fp_text reference J2 (at 1.27 8.255 90) (layer F.SilkS)
-      (effects (font (size 1 1) (thickness 0.15)))
+    (fp_text reference J2 (at 1.27 3.175 270) (layer B.SilkS)
+      (effects (font (size 1 1) (thickness 0.15)) (justify mirror))
     )
-    (fp_text value Conn_PinHeader_PCB (at -5.08 1.27 180) (layer F.Fab) hide
-      (effects (font (size 1 1) (thickness 0.15)))
+    (fp_text value Conn_PinHeader_PCB (at -5.08 -1.27 180) (layer B.Fab) hide
+      (effects (font (size 1 1) (thickness 0.15)) (justify mirror))
     )
-    (fp_text user %R (at 1.27 2.54) (layer F.Fab)
-      (effects (font (size 1 1) (thickness 0.15)))
+    (fp_text user %R (at 1.27 -2.54) (layer B.Fab)
+      (effects (font (size 1 1) (thickness 0.15)) (justify mirror))
     )
-    (fp_line (start 4.35 -1.8) (end -1.8 -1.8) (layer F.CrtYd) (width 0.05))
-    (fp_line (start 4.35 6.85) (end 4.35 -1.8) (layer F.CrtYd) (width 0.05))
-    (fp_line (start -1.8 6.85) (end 4.35 6.85) (layer F.CrtYd) (width 0.05))
-    (fp_line (start -1.8 -1.8) (end -1.8 6.85) (layer F.CrtYd) (width 0.05))
-    (fp_line (start -1.33 -1.33) (end 0 -1.33) (layer F.SilkS) (width 0.12))
-    (fp_line (start -1.33 0) (end -1.33 -1.33) (layer F.SilkS) (width 0.12))
-    (fp_line (start 1.27 -1.33) (end 3.87 -1.33) (layer F.SilkS) (width 0.12))
-    (fp_line (start 1.27 1.27) (end 1.27 -1.33) (layer F.SilkS) (width 0.12))
-    (fp_line (start -1.33 1.27) (end 1.27 1.27) (layer F.SilkS) (width 0.12))
-    (fp_line (start 3.87 -1.33) (end 3.87 6.41) (layer F.SilkS) (width 0.12))
-    (fp_line (start -1.33 1.27) (end -1.33 6.41) (layer F.SilkS) (width 0.12))
-    (fp_line (start -1.33 6.41) (end 3.87 6.41) (layer F.SilkS) (width 0.12))
-    (fp_line (start -1.27 0) (end 0 -1.27) (layer F.Fab) (width 0.1))
-    (fp_line (start -1.27 6.35) (end -1.27 0) (layer F.Fab) (width 0.1))
-    (fp_line (start 3.81 6.35) (end -1.27 6.35) (layer F.Fab) (width 0.1))
-    (fp_line (start 3.81 -1.27) (end 3.81 6.35) (layer F.Fab) (width 0.1))
-    (fp_line (start 0 -1.27) (end 3.81 -1.27) (layer F.Fab) (width 0.1))
-    (pad 4 thru_hole oval (at 2.54 5.08 270) (size 1.7 1.7) (drill 1) (layers *.Cu *.Mask)
+    (fp_line (start 4.35 1.8) (end -1.8 1.8) (layer B.CrtYd) (width 0.05))
+    (fp_line (start 4.35 -6.85) (end 4.35 1.8) (layer B.CrtYd) (width 0.05))
+    (fp_line (start -1.8 -6.85) (end 4.35 -6.85) (layer B.CrtYd) (width 0.05))
+    (fp_line (start -1.8 1.8) (end -1.8 -6.85) (layer B.CrtYd) (width 0.05))
+    (fp_line (start -1.33 1.33) (end 0 1.33) (layer B.SilkS) (width 0.12))
+    (fp_line (start -1.33 0) (end -1.33 1.33) (layer B.SilkS) (width 0.12))
+    (fp_line (start 1.27 1.33) (end 3.87 1.33) (layer B.SilkS) (width 0.12))
+    (fp_line (start 1.27 -1.27) (end 1.27 1.33) (layer B.SilkS) (width 0.12))
+    (fp_line (start -1.33 -1.27) (end 1.27 -1.27) (layer B.SilkS) (width 0.12))
+    (fp_line (start 3.87 1.33) (end 3.87 -6.41) (layer B.SilkS) (width 0.12))
+    (fp_line (start -1.33 -1.27) (end -1.33 -6.41) (layer B.SilkS) (width 0.12))
+    (fp_line (start -1.33 -6.41) (end 3.87 -6.41) (layer B.SilkS) (width 0.12))
+    (fp_line (start -1.27 0) (end 0 1.27) (layer B.Fab) (width 0.1))
+    (fp_line (start -1.27 -6.35) (end -1.27 0) (layer B.Fab) (width 0.1))
+    (fp_line (start 3.81 -6.35) (end -1.27 -6.35) (layer B.Fab) (width 0.1))
+    (fp_line (start 3.81 1.27) (end 3.81 -6.35) (layer B.Fab) (width 0.1))
+    (fp_line (start 0 1.27) (end 3.81 1.27) (layer B.Fab) (width 0.1))
+    (pad 4 thru_hole oval (at 2.54 -5.08 270) (size 1.7 1.7) (drill 1) (layers *.Cu *.Mask)
       (net 5 "Net-(J1-Pad5)"))
-    (pad 3 thru_hole oval (at 0 5.08 270) (size 1.7 1.7) (drill 1) (layers *.Cu *.Mask)
+    (pad 3 thru_hole oval (at 0 -5.08 270) (size 1.7 1.7) (drill 1) (layers *.Cu *.Mask)
       (net 1 "Net-(J1-Pad1)"))
-    (pad 5 thru_hole oval (at 2.54 2.54 270) (size 1.7 1.7) (drill 1) (layers *.Cu *.Mask)
+    (pad 5 thru_hole oval (at 2.54 -2.54 270) (size 1.7 1.7) (drill 1) (layers *.Cu *.Mask)
       (net 5 "Net-(J1-Pad5)"))
-    (pad 2 thru_hole oval (at 0 2.54 270) (size 1.7 1.7) (drill 1) (layers *.Cu *.Mask)
+    (pad 2 thru_hole oval (at 0 -2.54 270) (size 1.7 1.7) (drill 1) (layers *.Cu *.Mask)
       (net 1 "Net-(J1-Pad1)"))
     (pad 6 thru_hole oval (at 2.54 0 270) (size 1.7 1.7) (drill 1) (layers *.Cu *.Mask)
@@
       (net 1 "Net-(J1-Pad1)"))
     (model ${KISYS3DMOD}/Connector_PinHeader_2.54mm.3dshapes/PinHeader_2x03_P2.54mm_Vertical.wrl
-      (offset (xyz 2.54 0 -2))
+      (at (xyz 0 0 0))
       (scale (xyz 1 1 1))
-      (rotate (xyz 0 180 0))
+      (rotate (xyz 0 0 0))
     )
   )
