File: logical-probe-1/logical-probe-1.kicad_pcb (KiCad board)
At the start: 2 copper layers, 129.5 x 25.4 mm, 14 parts, among them J1 VDD, J2 Probe, U1 4001

Commit message: update: update footprints & Gerber files
Parts:
- J2: footprint logical-probe-1:probe_1mm -> logical-probe-1:probe_1mm_pcb
Routing:
- net Signal-in: track 52.9 -> 61.0 mm
- added copper zone on B.Cu, net Signal-in
