File: logical-probe-1/logical-probe-1.sch (KiCad schematic (older format))
At the start: 13 parts, among them J1 VDD, J2 Probe, U1 4001

Commit message: update: update footprints & Gerber files
Parts:
- J2: footprint logical-probe-1:probe_1mm -> logical-probe-1:probe_1mm_pcb
Changed lines of the file:
@@
 F 0 "J2" H 9730 4542 50  0000 L CNN
 F 1 "Probe" H 9730 4451 50  0000 L CNN
-F 2 "logical-probe-1:probe_1mm" H 9650 4500 50  0001 C CNN
+F 2 "logical-probe-1:probe_1mm_pcb" H 9650 4500 50  0001 C CNN
 F 3 "~" H 9650 4500 50  0001 C CNN
 	1    9650 4500
